File: PCB Schemas/Square/square.sch (EAGLE design)
At the start: 10 parts

Commit message: Updated and Finalized Square Board V1
Parts:
- removed JP1: (no value), pinhead:PINHD-1X5
- added J1: CON_5P_1.27, Connectors:CON_5P_1.27
- R2: value 220 -> 10k
- R3: value 10k -> 220
Connections:
- net COLOR: now also J1-3.S, R2.1; no longer JP1.3, R3.1
- net G: now also J1-5.S; no longer JP1.5
- net GND: now also J1-2.S, R3.1; no longer JP1.2, R1.1
- net N$1: now also R3.2; no longer R1.2
- net N$2: now also R1.2; no longer R2.2
- net R: now also J1-4.S; no longer JP1.4
- net VCC: now also J1-1.S, R1.1, R2.2; no longer JP1.1, R2.1, R3.2
Other:
- moved on the sheet: R1, R2, R3
Changed lines of the file:
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@@
 <setting verticaltext="up"/>
 </settings>
-<grid distance="0.1" unitdist="inch" unit="inch" style="lines" multiple="1" display="no" altdistance="0.01" altunitdist="inch" altunit="inch"/>
+<grid distance="0.1" unitdist="inch" unit="mm" style="lines" multiple="1" display="no" altdistance="0.01" altunitdist="inch" altunit="inch"/>
 <layers>
 <layer number="1" name="Top" color="4" fill="1" visible="no" active="no"/>
@@
 <parts>
 <part name="LED1" library="led" deviceset="L-115WEGW-CA" device="" value=""/>
-<part name="R1" library="resistor" deviceset="R-EU_" device="0204/7" value="220"/>
+<part name="R3" library="resistor" deviceset="R-EU_" device="0204/7" value="220"/>
 <part name="GND4" library="supply1" deviceset="GND" device=""/>
 <part name="GND5" library="supply1" deviceset="GND" device=""/>
 <part name="P+1" library="supply1" deviceset="VCC" device=""/>
 <part name="P+3" library="supply1" deviceset="VCC" device=""/>
-<part name="R2" library="resistor" deviceset="R-EU_" device="0204/7" value="220"/>
-<part name="R3" library="resistor" deviceset="R-EU_" device="0204/7" value="10k"/>
+<part name="R1" library="resistor" deviceset="R-EU_" device="0204/7" value="220"/>
+<part name="R2" library="resistor" deviceset="R-EU_" device="0204/7" value="10k"/>
 <part name="LED2" library="led" deviceset="L-115WEGW-CA" device="" value=""/>
 <part name="LED3" library="led" deviceset="L-115WEGW-CA" device="" value=""/>
@@
 <part name="GND8" library="supply1" deviceset="GND" device=""/>
 <part name="GND1" library="supply1" deviceset="GND" device=""/>
-<part name="JP1" library="pinhead" deviceset="PINHD-1X5" device=""/>
 <part name="P+2" library="supply1" deviceset="VCC" device=""/>
 <part name="GND2" library="supply1" deviceset="GND" device=""/>
 <part name="CNY70" library="cny70" deviceset="CNY70" device="" value=""/>
+<part name="J1" library="Connectors" deviceset="CON_5P_1.27" device="" value=""/>
 </parts>
 <sheets>
@@
 <instances>
 <instance part="LED1" gate="G$1" x="40.64" y="50.8"/>
-<instance part="R1" gate="G$1" x="27.94" y="50.8"/>
+<instance part="R3" gate="G$1" x="27.94" y="50.8"/>
 <instance part="GND4" gate="1" x="17.78" y="50.8" rot="R270"/>
 <instance part="GND5" gate="1" x="20.32" y="68.58" rot="R270"/>
 <instance part="P+1" gate="VCC" x="2.54" y="76.2"/>
 <instance part="P+3" gate="VCC" x="60.96" y="76.2"/>
-<instance part="R2" gate="G$1" x="15.24" y="73.66"/>
-<instance part="R3" gate="G$1" x="53.34" y="73.66"/>
+<instance part="R1" gate="G$1" x="15.24" y="73.66"/>
+<instance part="R2" gate="G$1" x="53.34" y="73.66"/>
 <instance part="LED2" gate="G$1" x="40.64" y="33.02"/>
 <instance part="LED3" gate="G$1" x="40.64" y="15.24"/>
@@
 <instance part="GND8" gate="1" x="17.78" y="15.24" rot="R270"/>
 <instance part="GND1" gate="1" x="43.18" y="68.58" rot="R90"/>
-<instance part="JP1" gate="A" x="116.84" y="38.1"/>
 <instance part="P+2" gate="VCC" x="99.06" y="45.72"/>
 <instance part="GND2" gate="1" x="99.06" y="40.64" rot="R270"/>
 <instance part="CNY70" gate="G$1" x="33.02" y="71.12"/>
+<instance part="J1" gate="-1" x="116.84" y="43.18"/>
+<instance part="J1" gate="-2" x="116.84" y="40.64"/>
+<instance part="J1" gate="-3" x="116.84" y="38.1"/>
+<instance part="J1" gate="-4" x="116.84" y="35.56"/>
+<instance part="J1" gate="-5" x="116.84" y="33.02"/>
 </instances>
 <busses>
@@
 <net name="N$1" class="0">
 <segment>
-<pinref part="R1" gate="G$1" pin="2"/>
+<pinref part="R3" gate="G$1" pin="2"/>
 <pinref part="LED1" gate="G$1" pin="A"/>
 <wire x1="33.02" y1="50.8" x2="38.1" y2="50.8" width="0.1524" layer="91"/>
@@
 <net name="GND" class="0">
 <segment>
-<pinref part="R1" gate="G$1" pin="1"/>
+<pinref part="R3" gate="G$1" pin="1"/>
 <pinref part="GND4" gate="1" pin="GND"/>
 <wire x1="22.86" y1="50.8" x2="20.32" y2="50.8" width="0.1524" layer="91"/>
@@
 </segment>
 <segment>
-<pinref part="JP1" gate="A" pin="2"/>
 <pinref part="GND2" gate="1" pin="GND"/>
 <wire x1="114.3" y1="40.64" x2="101.6" y2="40.64" width="0.1524" layer="91"/>
+<pinref part="J1" gate="-2" pin="S"/>
 </segment>
 <segment>
@@
 <net name="N$2" class="0">
 <segment>
-<pinref part="R2" gate="G$1" pin="2"/>
+<pinref part="R1" gate="G$1" pin="2"/>
 <wire x1="22.86" y1="73.66" x2="20.32" y2="73.66" width="0.1524" layer="91"/>
 <pinref part="CNY70" gate="G$1" pin="A"/>
@@
 <segment>
 <pinref part="P+1" gate="VCC" pin="VCC"/>
-<pinref part="R2" gate="G$1" pin="1"/>
+<pinref part="R1" gate="G$1" pin="1"/>
 <wire x1="2.54" y1="73.66" x2="10.16" y2="73.66" width="0.1524" layer="91"/>
 </segment>
 <segment>
-<pinref part="R3" gate="G$1" pin="2"/>
+<pinref part="R2" gate="G$1" pin="2"/>
 <pinref part="P+3" gate="VCC" pin="VCC"/>
 <wire x1="58.42" y1="73.66" x2="60.96" y2="73.66" width="0.1524" layer="91"/>
 </segment>
 <segment>
-<pinref part="JP1" gate="A" pin="1"/>
 <pinref part="P+2" gate="VCC" pin="VCC"/>
 <wire x1="114.3" y1="43.18" x2="99.06" y2="43.18" width="0.1524" layer="91"/>
+<pinref part="J1" gate="-1" pin="S"/>
 </segment>
 </net>
@@
 </segment>
 <segment>
-<pinref part="JP1" gate="A" pin="4"/>
 <wire x1="114.3" y1="35.56" x2="104.14" y2="35.56" width="0.1524" layer="91"/>
 <label x="104.14" y="35.56" size="1.778" layer="95"/>
+<pinref part="J1" gate="-4" pin="S"/>
 </segment>
 </net>
@@
 </segment>
 <segment>
-<pinref part="JP1" gate="A" pin="5"/>
 <wire x1="114.3" y1="33.02" x2="104.14" y2="33.02" width="0.1524" layer="91"/>
 <label x="104.14" y="33.02" size="1.778" layer="95"/>
+<pinref part="J1" gate="-5" pin="S"/>
 </segment>
 </net>
@@
 <label x="40.64" y="81.28" size="1.778" layer="95"/>
 <wire x1="40.64" y1="73.66" x2="48.26" y2="73.66" width="0.1524" layer="91"/>
-<pinref part="R3" gate="G$1" pin="1"/>
+<pinref part="R2" gate="G$1" pin="1"/>
 <pinref part="CNY70" gate="G$1" pin="COL"/>
 </segment>
 <segment>
-<pinref part="JP1" gate="A" pin="3"/>
 <wire x1="114.3" y1="38.1" x2="104.14" y2="38.1" width="0.1524" layer="91"/>
 <label x="104.14" y="38.1" size="1.778" layer="95"/>
-</segment>
-</net>
+<pinref part="J1" gate="-3" pin="S"/>
+</segment>
+</net>
