File: PCB Schemas/BaseBoard/BaseBoard.brd (EAGLE design)
At the start: 100 x 80 mm, 28 parts, among them IC1 74HC595N, IC2 74HC595N, IC3 74HC595N, Q1 16MHz, U1 ATMEGA2560AU, X1 SQUARE1, X2 SQUARE2, X3 SQUARE3, X4 SQUARE4, X5 53261-05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

Commit message: completed the schema, still need to add the comm bus
Parts:
- X5: value 53261-05 -> SQUARE5
- X6: value 53261-05 -> SQUARE6
- X7: value 53261-05 -> SQUARE7
- X8: value 53261-05 -> SQUARE8
- X9: value 53261-05 -> SQUARE9
Connections:
- new net COL4: U1.94, X4.3
- new net COL5: U1.93, X5.3
- new net COL6: U1.92, X6.3
- new net COL7: U1.91, X7.3
- new net GRE4: IC2.15, X4.4
- new net GRE5: IC2.2, X5.4
- new net GRE6: IC2.4, X6.4
- new net GRE7: IC3.15, X7.4
- new net GRE8: IC3.2, X8.4
- new net GRE9: IC3.4, X9.4
- new net N$28: IC3.13
- new net RED4: IC2.1, X4.5
- new net RED5: IC2.3, X5.5
- new net RED6: X6.5
- new net RED7: IC3.1, X7.5
- new net RED8: IC3.3, X8.5
- new net RED9: IC3.5, X9.5
- net CLK: now also IC3.11
- net COL3: now also X3.3
- net COL8: now also X8.3
- net COL9: now also X9.3
- net GRE3: now also X3.4
- net LATCH: now also IC3.12
- net RED3: now also X3.5
- net VCC: now also IC1.10

Commit message: board still needs some work
Parts:
- removed U$1: LED_PIRANHA_5MM, SparkFun-LED:LED_PIRANHA_5MM
- added DEBUG_LED: LED_PIRANHA_5MM, SparkFun-LED:LED_PIRANHA_5MM
- moved R5 165.5 mm to (97.8, 12.7), turned to 270 degrees
- moved C3 156.3 mm to (86.4, 8.89), turned to 180 degrees
- moved JP1 151.4 mm to (86.4, 1.27)
- moved LED1 147.4 mm to (77.5, 14.0)
- moved R4 144.8 mm to (86.4, 14.0)
- moved C2 139.0 mm to (92.7, 19.1)
- moved R2 136.3 mm to (95.2, 8.89), turned to 90 degrees
- moved R3 131.3 mm to (77.5, 5.08), turned to 90 degrees
- moved C1 123.7 mm to (85.1, 21.6), turned to 90 degrees
- moved Q1 111.9 mm to (92.7, 29.2)
- moved X4 111.5 mm to (87.6, 72.4)
- moved X5 111.5 mm to (73.7, 72.4)
- moved X6 111.5 mm to (59.7, 72.4)
- moved IC2 101.2 mm to (71.1, 58.4), turned to 180 degrees
- moved C5 100.1 mm to (73.7, 40.6), turned to 180 degrees
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Connections:
- net DBG_B: now also DEBUG_LED.B; no longer U$1.B
- net DBG_G: now also DEBUG_LED.G; no longer U$1.G
- net DBG_R: now also DEBUG_LED.R; no longer U$1.R
- net N$9: now also DEBUG_LED.-; no longer U$1.-

Commit message: changed schema and board
Parts:
- X1: value SQUARE1 -> SQU1
- X2: value SQUARE2 -> SQU2
- X3: value SQUARE3 -> SQU3
- X4: value SQUARE4 -> SQU4
- X5: value SQUARE5 -> SQU5
- X6: value SQUARE6 -> SQU6
- X7: value SQUARE7 -> SQU7
- X8: value SQUARE8 -> SQU8
- X9: value SQUARE9 -> SQU9
- moved R5 35.8 mm to (94.0, 48.3), turned to 180 degrees
- moved R4 34.4 mm to (83.8, 48.3)
- moved DEBUG_LED 4.58 mm to (88.9, 36.8)
Changed lines of the file:
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@@
 <element name="C5" library="capacitor-wima" package="C5B3" value="100nF" x="73.66" y="40.64" rot="R180"/>
 <element name="JP2" library="SparkFun-Connectors" package="1X02" value="M02PTH" x="1.27" y="33.02" rot="R270"/>
-<element name="X1" library="con-molex" package="53261-05" value="SQUARE1" x="45.72" y="72.39">
+<element name="X1" library="con-molex" package="53261-05" value="SQU1" x="45.72" y="72.39">
 <attribute name="OC_NEWARK" value="unknown" x="77.47" y="38.1" size="1.778" layer="27" display="off"/>
 <attribute name="MPN" value="" x="77.47" y="38.1" size="1.778" layer="27" display="off"/>
@@
 <attribute name="OC_FARNELL" value="1433644" x="77.47" y="38.1" size="1.778" layer="27" display="off"/>
 </element>
-<element name="X2" library="con-molex" package="53261-05" value="SQUARE2" x="30.48" y="72.39">
+<element name="X2" library="con-molex" package="53261-05" value="SQU2" x="30.48" y="72.39">
 <attribute name="OC_NEWARK" value="unknown" x="76.2" y="38.1" size="1.778" layer="27" display="off"/>
 <attribute name="MPN" value="" x="76.2" y="38.1" size="1.778" layer="27" display="off"/>
@@
 <attribute name="OC_FARNELL" value="1433644" x="76.2" y="38.1" size="1.778" layer="27" display="off"/>
 </element>
-<element name="X3" library="con-molex" package="53261-05" value="SQUARE3" x="16.51" y="72.39">
+<element name="X3" library="con-molex" package="53261-05" value="SQU3" x="16.51" y="72.39">
 <attribute name="OC_NEWARK" value="unknown" x="76.2" y="38.1" size="1.778" layer="27" display="off"/>
 <attribute name="MPN" value="" x="76.2" y="38.1" size="1.778" layer="27" display="off"/>
@@
 <attribute name="OC_FARNELL" value="1433644" x="76.2" y="38.1" size="1.778" layer="27" display="off"/>
 </element>
-<element name="X4" library="con-molex" package="53261-05" value="SQUARE4" x="87.63" y="72.39">
+<element name="X4" library="con-molex" package="53261-05" value="SQU4" x="87.63" y="72.39">
 <attribute name="OC_NEWARK" value="unknown" x="107.95" y="27.94" size="1.778" layer="27" display="off"/>
 <attribute name="MPN" value="" x="107.95" y="27.94" size="1.778" layer="27" display="off"/>
@@
 <attribute name="OC_FARNELL" value="1433644" x="107.95" y="27.94" size="1.778" layer="27" display="off"/>
 </element>
-<element name="X5" library="con-molex" package="53261-05" value="SQUARE5" x="73.66" y="72.39">
+<element name="X5" library="con-molex" package="53261-05" value="SQU5" x="73.66" y="72.39">
 <attribute name="OC_NEWARK" value="unknown" x="107.95" y="27.94" size="1.778" layer="27" display="off"/>
 <attribute name="MPN" value="" x="107.95" y="27.94" size="1.778" layer="27" display="off"/>
@@
 <attribute name="OC_FARNELL" value="1433644" x="107.95" y="27.94" size="1.778" layer="27" display="off"/>
 </element>
-<element name="X6" library="con-molex" package="53261-05" value="SQUARE6" x="59.69" y="72.39">
+<element name="X6" library="con-molex" package="53261-05" value="SQU6" x="59.69" y="72.39">
 <attribute name="OC_NEWARK" value="unknown" x="107.95" y="27.94" size="1.778" layer="27" display="off"/>
 <attribute name="MPN" value="" x="107.95" y="27.94" size="1.778" layer="27" display="off"/>
@@
 <attribute name="OC_FARNELL" value="1433644" x="107.95" y="27.94" size="1.778" layer="27" display="off"/>
 </element>
-<element name="X7" library="con-molex" package="53261-05" value="SQUARE7" x="21.59" y="8.89" rot="R180">
+<element name="X7" library="con-molex" package="53261-05" value="SQU7" x="21.59" y="8.89" rot="R180">
 <attribute name="OC_NEWARK" value="unknown" x="-40.64" y="53.34" size="1.778" layer="27" rot="R180" display="off"/>
 <attribute name="MPN" value="" x="-40.64" y="53.34" size="1.778" layer="27" rot="R180" display="off"/>
@@
 <attribute name="OC_FARNELL" value="1433644" x="-40.64" y="53.34" size="1.778" layer="27" rot="R180" display="off"/>
 </element>
-<element name="X8" library="con-molex" package="53261-05" value="SQUARE8" x="35.56" y="8.89" rot="R180">
+<element name="X8" library="con-molex" package="53261-05" value="SQU8" x="35.56" y="8.89" rot="R180">
 <attribute name="OC_NEWARK" value="unknown" x="15.24" y="62.23" size="1.778" layer="27" rot="R180" display="off"/>
 <attribute name="MPN" value="" x="15.24" y="62.23" size="1.778" layer="27" rot="R180" display="off"/>
@@
 <attribute name="OC_FARNELL" value="1433644" x="15.24" y="62.23" size="1.778" layer="27" rot="R180" display="off"/>
 </element>
-<element name="X9" library="con-molex" package="53261-05" value="SQUARE9" x="49.53" y="8.89" rot="R180">
+<element name="X9" library="con-molex" package="53261-05" value="SQU9" x="49.53" y="8.89" rot="R180">
 <attribute name="OC_NEWARK" value="unknown" x="15.24" y="62.23" size="1.778" layer="27" rot="R180" display="off"/>
 <attribute name="MPN" value="" x="15.24" y="62.23" size="1.778" layer="27" rot="R180" display="off"/>
@@
 <element name="IC3" library="74xx-eu" package="DIL16" value="74HC595N" x="40.64" y="22.86"/>
 <element name="LED1" library="SparkFun-LED" package="LED3MM" value="" x="77.47" y="13.97"/>
-<element name="DEBUG_LED" library="SparkFun-LED" package="LED_PIRANHA_5MM" value="LED_PIRANHA_5MM" x="92.71" y="39.37" rot="R180"/>
-<element name="R4" library="resistor" package="0204/7" value="330" x="86.36" y="13.97"/>
-<element name="R5" library="resistor" package="0204/7" value="330" x="97.79" y="12.7" rot="R270"/>
+<element name="DEBUG_LED" library="SparkFun-LED" package="LED_PIRANHA_5MM" value="LED_PIRANHA_5MM" x="88.9" y="36.83" rot="R180"/>
+<element name="R4" library="resistor" package="0204/7" value="330" x="83.82" y="48.26"/>
+<element name="R5" library="resistor" package="0204/7" value="330" x="93.98" y="48.26" rot="R180"/>
 </elements>
 <signals>
@@
 <wire x1="85.09" y1="19.05" x2="76.2" y2="40.64" width="0" layer="19" extent="1-1"/>
 <wire x1="90.17" y1="19.05" x2="85.09" y2="19.05" width="0" layer="19" extent="1-1"/>
-<wire x1="90.17" y1="13.97" x2="90.17" y2="19.05" width="0" layer="19" extent="1-1"/>
-<wire x1="97.79" y1="8.89" x2="90.17" y2="13.97" width="0" layer="19" extent="1-1"/>
-<wire x1="86.36" y1="1.27" x2="97.79" y2="8.89" width="0" layer="19" extent="1-1"/>
+<wire x1="87.63" y1="48.26" x2="90.17" y2="19.05" width="0" layer="19" extent="1-1"/>
+<wire x1="90.17" y1="48.26" x2="87.63" y2="48.26" width="0" layer="19" extent="1-1"/>
+<wire x1="86.36" y1="1.27" x2="90.17" y2="48.26" width="0" layer="19" extent="1-1"/>
 <wire x1="1.27" y1="33.02" x2="86.36" y2="1.27" width="0" layer="19" extent="1-1"/>
 <wire x1="34.31" y1="11.39" x2="76.2" y2="46.99" width="0" layer="19" extent="1-1"/>
@@
 <contactref element="LED1" pad="K"/>
 <contactref element="R4" pad="1"/>
-<wire x1="78.74" y1="13.97" x2="82.55" y2="13.97" width="0" layer="19" extent="1-1"/>
+<wire x1="78.74" y1="13.97" x2="80.01" y2="48.26" width="0" layer="19" extent="1-1"/>
 </signal>
 <signal name="N$9">
 <contactref element="DEBUG_LED" pad="-"/>
 <contactref element="R5" pad="1"/>
-<wire x1="95.394" y1="42.054" x2="97.79" y2="16.51" width="0" layer="19" extent="1-1"/>
+<wire x1="91.584" y1="39.514" x2="97.79" y2="48.26" width="0" layer="19" extent="1-1"/>
 </signal>
 <signal name="DBG_R">
 <contactref element="DEBUG_LED" pad="R"/>
 <contactref element="U1" pad="53"/>
-<wire x1="90.131" y1="42.066" x2="43.26" y2="33.91" width="0" layer="19" extent="1-1"/>
+<wire x1="86.321" y1="39.526" x2="43.26" y2="33.91" width="0" layer="19" extent="1-1"/>
 </signal>
 <signal name="DBG_B">
 <contactref element="DEBUG_LED" pad="B"/>
 <contactref element="U1" pad="54"/>
-<wire x1="95.398" y1="36.796" x2="43.76" y2="33.91" width="0" layer="19" extent="1-1"/>
+<wire x1="91.588" y1="34.256" x2="43.76" y2="33.91" width="0" layer="19" extent="1-1"/>
 </signal>
 <signal name="DBG_G">
 <contactref element="DEBUG_LED" pad="G"/>
 <contactref element="U1" pad="55"/>
-<wire x1="44.26" y1="33.91" x2="90.135" y2="36.808" width="0" layer="19" extent="1-1"/>
+<wire x1="44.26" y1="33.91" x2="86.325" y2="34.268" width="0" layer="19" extent="1-1"/>
 </signal>
 <signal name="GRE4">
