File: PCB Schemas/Square V1/square.brd (EAGLE design)
At the start: 38.4 x 38.1 mm, 10 parts

Commit message: Updated details
Parts:
- removed J1: (no value), Connectors:CON_5P_1.27
- added CON: (no value), Connectors:CON05_2.54MM
Connections:
- removed net G: J1.5, LED1.1, LED2.1, LED3.1
- removed net R: J1.4, LED1.3, LED2.3, LED3.3
- new net GREEN: CON.5, LED1.1, LED2.1, LED3.1
- new net RED: CON.4, LED1.3, LED2.3, LED3.3
- net COLOR: now also CON.3; no longer J1.3
- net GND: now also CON.2; no longer J1.2
- net VCC: now also CON.1; no longer J1.1
Routing:
- net GREEN: track 0.00 -> 67.9 mm
- net G: track 67.9 -> 0.00 mm
- net RED: track 0.00 -> 62.4 mm
- net R: track 62.4 -> 0.00 mm
Changed lines of the file:
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@@
 <?xml version="1.0" encoding="utf-8"?>
 <!DOCTYPE eagle SYSTEM "eagle.dtd">
-<eagle version="6.4">
+<eagle version="6.5.0">
 <drawing>
 <settings>
@@
 <attribute name="NAME" x="15.748" y="23.606" size="1.27" layer="25" ratio="10"/>
 </element>
-<element name="J1" library="Connectors" package="CON_5P_1.27" value="" x="19.05" y="3.81"/>
+<element name="CON" library="Connectors" package="CON05_2.54MM" value="" x="19.05" y="3.81" smashed="yes">
+<attribute name="NAME" x="16.8275" y="5.08" size="1.27" layer="21"/>
+<attribute name="VALUE" x="15.5575" y="1.27" size="1.27" layer="21"/>
+</element>
 </elements>
 <signals>
@@
 <wire x1="17.78" y1="10.16" x2="21.59" y2="10.16" width="0.4064" layer="16"/>
 <wire x1="20.32" y1="20.32" x2="17.78" y2="17.78" width="0.4064" layer="16"/>
-<contactref element="J1" pad="2"/>
 <wire x1="17.78" y1="17.78" x2="17.78" y2="10.16" width="0.4064" layer="16"/>
 <wire x1="11.43" y1="19.685" x2="13.335" y2="17.78" width="0.4064" layer="16"/>
@@
 <wire x1="11.43" y1="28.575" x2="11.43" y2="19.685" width="0.4064" layer="16"/>
 <wire x1="17.78" y1="3.81" x2="17.78" y2="17.78" width="0.4064" layer="16"/>
+<contactref element="CON" pad="2"/>
 </signal>
 <signal name="N$2">
@@
 <contactref element="R2" pad="2"/>
 <wire x1="12.065" y1="13.335" x2="15.24" y2="13.335" width="0.4064" layer="16"/>
-<contactref element="J1" pad="1"/>
 <wire x1="6.35" y1="20.32" x2="6.35" y2="19.05" width="0.4064" layer="16"/>
 <wire x1="6.35" y1="19.05" x2="12.065" y2="13.335" width="0.4064" layer="16"/>
@@
 <wire x1="16.51" y1="5.08" x2="15.24" y2="6.35" width="0.4064" layer="16"/>
 <wire x1="15.24" y1="6.35" x2="15.24" y2="13.335" width="0.4064" layer="16"/>
-</signal>
-<signal name="R">
+<contactref element="CON" pad="1"/>
+</signal>
+<signal name="RED">
 <contactref element="LED1" pad="3"/>
 <contactref element="LED2" pad="3"/>
 <contactref element="LED3" pad="3"/>
-<contactref element="J1" pad="4"/>
 <wire x1="20.32" y1="3.81" x2="20.32" y2="5.715" width="0.4064" layer="16"/>
 <wire x1="20.32" y1="5.715" x2="24.765" y2="10.16" width="0.4064" layer="16"/>
@@
 <wire x1="20.32" y1="3.81" x2="20.32" y2="2.54" width="0.4064" layer="16"/>
 <wire x1="20.32" y1="2.54" x2="19.685" y2="1.905" width="0.4064" layer="16"/>
-</signal>
-<signal name="G">
+<contactref element="CON" pad="4"/>
+</signal>
+<signal name="GREEN">
 <contactref element="LED1" pad="1"/>
 <contactref element="LED2" pad="1"/>
 <contactref element="LED3" pad="1"/>
-<contactref element="J1" pad="5"/>
 <wire x1="3.81" y1="12.359703125" x2="3.81" y2="22.86" width="0.4064" layer="16"/>
 <wire x1="3.81" y1="22.86" x2="16.51" y2="35.56" width="0.4064" layer="16"/>
@@
 <wire x1="21.59" y1="3.81" x2="21.59" y2="2.54" width="0.4064" layer="16"/>
 <wire x1="21.59" y1="2.54" x2="20.0025" y2="0.9525" width="0.4064" layer="16"/>
+<contactref element="CON" pad="5"/>
 </signal>
 <signal name="COLOR">
@@
 <wire x1="22.86" y1="13.335" x2="22.86" y2="15.24" width="0.4064" layer="16"/>
 <wire x1="22.86" y1="15.24" x2="20.32" y2="17.78" width="0.4064" layer="16"/>
-<contactref element="J1" pad="3"/>
 <wire x1="22.86" y1="13.335" x2="22.86" y2="9.525" width="0.4064" layer="16"/>
 <wire x1="22.86" y1="9.525" x2="19.05" y2="5.715" width="0.4064" layer="16"/>
 <wire x1="19.05" y1="5.715" x2="19.05" y2="3.81" width="0.4064" layer="16"/>
+<contactref element="CON" pad="3"/>
 </signal>
 </signals>
