File: PCB Schemas/Square V1/square.sch (EAGLE design)
At the start: 10 parts, among them J1 CON_5P_1.27

Commit message: Updated details
Parts:
- removed J1: CON_5P_1.27, Connectors:CON_5P_1.27
- added CON: CON05, Connectors:CON05
Connections:
- removed net G: J1-5.S, LED1.CG, LED2.CG, LED3.CG
- removed net R: J1-4.S, LED1.CR, LED2.CR, LED3.CR
- new net GREEN: CON.5, LED1.CG, LED2.CG, LED3.CG
- new net RED: CON.4, LED1.CR, LED2.CR, LED3.CR
- net COLOR: now also CON.3; no longer J1-3.S
- net GND: now also CON.2; no longer J1-2.S
- net VCC: now also CON.1; no longer J1-1.S
Changed lines of the file:
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@@
 <?xml version="1.0" encoding="utf-8"?>
 <!DOCTYPE eagle SYSTEM "eagle.dtd">
-<eagle version="6.4">
+<eagle version="6.5.0">
 <drawing>
 <settings>
@@
 <part name="GND2" library="supply1" deviceset="GND" device=""/>
 <part name="CNY70" library="cny70" deviceset="CNY70" device="" value=""/>
-<part name="J1" library="Connectors" deviceset="CON_5P_1.27" device="" value=""/>
+<part name="CON" library="Connectors" deviceset="CON05" device="" value=""/>
 </parts>
 <sheets>
@@
 <instance part="GND8" gate="1" x="17.78" y="15.24" rot="R270"/>
 <instance part="GND1" gate="1" x="43.18" y="68.58" rot="R90"/>
-<instance part="P+2" gate="VCC" x="99.06" y="45.72"/>
-<instance part="GND2" gate="1" x="99.06" y="40.64" rot="R270"/>
+<instance part="P+2" gate="VCC" x="114.3" y="48.26"/>
+<instance part="GND2" gate="1" x="114.3" y="27.94"/>
 <instance part="CNY70" gate="G$1" x="33.02" y="71.12"/>
-<instance part="J1" gate="-1" x="116.84" y="43.18"/>
-<instance part="J1" gate="-2" x="116.84" y="40.64"/>
-<instance part="J1" gate="-3" x="116.84" y="38.1"/>
-<instance part="J1" gate="-4" x="116.84" y="35.56"/>
-<instance part="J1" gate="-5" x="116.84" y="33.02"/>
+<instance part="CON" gate="G$1" x="121.92" y="38.1"/>
 </instances>
 <busses>
@@
 <segment>
 <pinref part="GND2" gate="1" pin="GND"/>
-<wire x1="114.3" y1="40.64" x2="101.6" y2="40.64" width="0.1524" layer="91"/>
-<pinref part="J1" gate="-2" pin="S"/>
+<pinref part="CON" gate="G$1" pin="2"/>
+<wire x1="116.84" y1="40.64" x2="114.3" y2="40.64" width="0.1524" layer="91"/>
+<wire x1="114.3" y1="40.64" x2="114.3" y2="30.48" width="0.1524" layer="91"/>
 </segment>
 <segment>
@@
 <segment>
 <pinref part="P+2" gate="VCC" pin="VCC"/>
-<wire x1="114.3" y1="43.18" x2="99.06" y2="43.18" width="0.1524" layer="91"/>
-<pinref part="J1" gate="-1" pin="S"/>
-</segment>
-</net>
-<net name="R" class="0">
+<pinref part="CON" gate="G$1" pin="1"/>
+<wire x1="116.84" y1="43.18" x2="114.3" y2="43.18" width="0.1524" layer="91"/>
+<wire x1="114.3" y1="43.18" x2="114.3" y2="45.72" width="0.1524" layer="91"/>
+</segment>
+</net>
+<net name="RED" class="0">
 <segment>
 <pinref part="LED1" gate="G$1" pin="CR"/>
@@
 </segment>
 <segment>
-<wire x1="114.3" y1="35.56" x2="104.14" y2="35.56" width="0.1524" layer="91"/>
-<label x="104.14" y="35.56" size="1.778" layer="95"/>
-<pinref part="J1" gate="-4" pin="S"/>
-</segment>
-</net>
-<net name="G" class="0">
+<label x="111.76" y="35.56" size="1.778" layer="95" rot="MR0"/>
+<wire x1="116.84" y1="35.56" x2="109.22" y2="35.56" width="0.1524" layer="91"/>
+<pinref part="CON" gate="G$1" pin="4"/>
+</segment>
+</net>
+<net name="GREEN" class="0">
 <segment>
 <pinref part="LED1" gate="G$1" pin="CG"/>
@@
 </segment>
 <segment>
-<wire x1="114.3" y1="33.02" x2="104.14" y2="33.02" width="0.1524" layer="91"/>
-<label x="104.14" y="33.02" size="1.778" layer="95"/>
-<pinref part="J1" gate="-5" pin="S"/>
+<label x="111.76" y="33.02" size="1.778" layer="95" rot="MR0"/>
+<wire x1="116.84" y1="33.02" x2="109.22" y2="33.02" width="0.1524" layer="91"/>
+<pinref part="CON" gate="G$1" pin="5"/>
 </segment>
 </net>
@@
 </segment>
 <segment>
-<wire x1="114.3" y1="38.1" x2="104.14" y2="38.1" width="0.1524" layer="91"/>
-<label x="104.14" y="38.1" size="1.778" layer="95"/>
-<pinref part="J1" gate="-3" pin="S"/>
-</segment>
-</net>
+<label x="111.76" y="38.1" size="1.778" layer="95" rot="MR0"/>
+<wire x1="116.84" y1="38.1" x2="109.22" y2="38.1" width="0.1524" layer="91"/>
+<pinref part="CON" gate="G$1" pin="3"/>
+</segment>
+</net>
