File: PCB Schemas/Square V2/square.brd (EAGLE design)
At the start: 36.8 x 36.8 mm, 13 parts

Commit message: Revised PCB schemas
Changed lines of the file:
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@@
 <setting verticaltext="up"/>
 </settings>
-<grid distance="0.0125" unitdist="inch" unit="mm" style="lines" multiple="1" display="no" altdistance="0.025" altunitdist="inch" altunit="inch"/>
+<grid distance="0.025" unitdist="inch" unit="inch" style="lines" multiple="1" display="no" altdistance="0.025" altunitdist="inch" altunit="inch"/>
 <layers>
 <layer number="1" name="Top" color="4" fill="1" visible="yes" active="yes"/>
@@
 <board>
 <plain>
-<wire x1="0" y1="0" x2="36.8175" y2="0" width="0" layer="20"/>
-<wire x1="36.8175" y1="0" x2="36.8175" y2="36.82" width="0" layer="20"/>
-<wire x1="36.8175" y1="36.82" x2="0" y2="36.82" width="0" layer="20"/>
+<wire x1="0" y1="0" x2="36.8" y2="0" width="0" layer="20"/>
+<wire x1="36.8" y1="0" x2="36.8" y2="36.8" width="0" layer="20"/>
+<wire x1="36.8" y1="36.8" x2="0" y2="36.8" width="0" layer="20"/>
 <text x="10.16" y="5.3975" size="1.27" layer="25">Tictactoe Square V2
 THOFU@2013</text>
@@
 <hole x="34.29" y="2.54" drill="3.2"/>
 <hole x="34.29" y="34.29" drill="3.2"/>
-<wire x1="0" y1="36.83" x2="0" y2="36.82" width="0" layer="20"/>
 <text x="10.795" y="2.54" size="1.27" layer="25">1</text>
-<wire x1="0" y1="36.82" x2="0" y2="0" width="0" layer="20"/>
+<wire x1="0" y1="36.8" x2="0" y2="0" width="0" layer="20"/>
 </plain>
 <attributes>
@@
 </element>
 <element name="R7" library="resistor" package="0204/7" value="220" x="20.955" y="28.575" smashed="yes" rot="R270">
-<attribute name="NAME" x="18.7579" y="27.6225" size="0.9906" layer="25" ratio="10" rot="R270"/>
+<attribute name="NAME" x="22.2504" y="27.94" size="0.9906" layer="25" ratio="10" rot="R270"/>
 <attribute name="VALUE" x="20.4724" y="30.2006" size="0.9906" layer="27" ratio="10" rot="R270"/>
 </element>
@@
 <element name="R6" library="resistor" package="0204/7" value="120" x="29.845" y="18.415" rot="R90"/>
 <element name="R8" library="resistor" package="0204/7" value="120" x="15.875" y="28.575" smashed="yes" rot="R270">
-<attribute name="NAME" x="17.1704" y="27.6225" size="0.9906" layer="25" ratio="10" rot="R270"/>
+<attribute name="NAME" x="13.6779" y="27.94" size="0.9906" layer="25" ratio="10" rot="R270"/>
 <attribute name="VALUE" x="15.3924" y="30.2006" size="0.9906" layer="27" ratio="10" rot="R270"/>
 </element>
